Commit message: can launch robot in gazebo. need plugins

File: openDog_description/urdf/openDog_full.urdf (robot description, URDF)
Before this commit: robot openDog, 13 links, 12 joints
Links:
- link hip_tube_1: mass None -> 1; geometry collision cylinder length=0.165 radius=0.05715; visual cylinder length=0.165 radius=0.05715
- link hip_tube_2: mass None -> 1; geometry collision cylinder length=0.165 radius=0.05715; visual cylinder length=0.165 radius=0.05715
- link hip_tube_3: mass None -> 1; geometry collision cylinder length=0.165 radius=0.05715; visual cylinder length=0.165 radius=0.05715
- link hip_tube_4: mass None -> 1; geometry collision cylinder length=0.165 radius=0.05715; visual cylinder length=0.165 radius=0.05715
- link lower_extrusion_leg1: mass None -> 1; geometry collision box size=0.02 0.04 0.31; visual box size=0.02 0.04 0.31
- link lower_extrusion_leg2: mass None -> 1; geometry collision box size=0.02 0.04 0.31; visual box size=0.02 0.04 0.31
- link lower_extrusion_leg3: mass None -> 1; geometry collision box size=0.02 0.04 0.31; visual box size=0.02 0.04 0.31
- link lower_extrusion_leg4: mass None -> 1; geometry collision box size=0.02 0.04 0.31; visual box size=0.02 0.04 0.31
- link openDog_body: mass None -> 1; geometry collision box size=0.31 0.881 0.195; visual box size=0.31 0.881 0.195
- link upper_extrusion_leg1: mass None -> 1; geometry collision box size=0.02 0.06 0.39; visual box size=0.02 0.06 0.39
- link upper_extrusion_leg2: mass None -> 1; geometry collision box size=0.02 0.06 0.39; visual box size=0.02 0.06 0.39
- link upper_extrusion_leg3: mass None -> 1; geometry collision box size=0.02 0.06 0.39; visual box size=0.02 0.06 0.39
- link upper_extrusion_leg4: mass None -> 1; geometry collision box size=0.02 0.06 0.39; visual box size=0.02 0.06 0.39

Commit message: trying control plugin

File: openDog_description/urdf/openDog_full.urdf (robot description, URDF)
Before this commit: robot openDog, 13 links, 12 joints
Links:
- added link openDog_body2, mass 1
- link openDog_body: mass 1 -> None
Joints:
- added joint dummy_link: type fixed, parent openDog_body, child openDog_body2, origin xyz=0 0 0 rpy=0 0 0
