Commit message: joint angles are added. need to revise femur angle value

File: urdf/openDog_full.urdf (robot description, URDF)
Before this commit: robot openDog, 14 links, 13 joints
Joints:
- joint femur_joint1: limit lower=0 upper=0.44 effort=0.1 velocity=0.005 -> lower=0.567 upper=1.579 effort=10 velocity=10
- joint femur_joint2: limit lower=0 upper=0.44 effort=0.1 velocity=0.005 -> lower=0.567 upper=1.579 effort=10 velocity=10
- joint femur_joint3: limit lower=0 upper=0.44 effort=0.1 velocity=0.005 -> lower=0.567 upper=1.579 effort=10 velocity=10
- joint femur_joint4: limit lower=0 upper=0.44 effort=0.1 velocity=0.005 -> lower=0.567 upper=1.579 effort=10 velocity=10
- joint knee_joint_leg1: limit lower=-2.2 upper=0.7 effort=30 velocity=1.0 -> lower=1.352 upper=2.8715 effort=10 velocity=10
- joint knee_joint_leg2: limit lower=-2.2 upper=0.7 effort=30 velocity=1.0 -> lower=1.352 upper=2.8715 effort=10 velocity=10
- joint knee_joint_leg3: limit lower=-2.2 upper=0.7 effort=30 velocity=1.0 -> lower=1.352 upper=2.8715 effort=10 velocity=10
- joint knee_joint_leg4: axis 0 1 0 -> 0 0 1; limit lower=-2.2 upper=0.7 effort=30 velocity=1.0 -> lower=1.352 upper=2.8715 effort=10 velocity=10

Commit message: need to debug leg angle limits

File: urdf/openDog_full.urdf (robot description, URDF)
Before this commit: robot openDog, 14 links, 13 joints
Joints:
- joint femur_joint1: limit lower=0.567 upper=1.579 effort=10 velocity=10 -> lower=-0.567 upper=-1.579 effort=10 velocity=10
- joint femur_joint2: limit lower=0.567 upper=1.579 effort=10 velocity=10 -> lower=-0.567 upper=-1.579 effort=10 velocity=10
- joint femur_joint3: limit lower=0.567 upper=1.579 effort=10 velocity=10 -> lower=-0.567 upper=-1.579 effort=10 velocity=10
- joint femur_joint4: limit lower=0.567 upper=1.579 effort=10 velocity=10 -> lower=-0.567 upper=-1.579 effort=10 velocity=10

Commit message: ros controller package added

File: urdf/openDog_full.urdf (robot description, URDF)
Before this commit: robot openDog, 14 links, 13 joints
Joints:
- joint femur_joint1: limit lower=-0.567 upper=-1.579 effort=10 velocity=10 -> lower=-1.579 upper=-0.567 effort=10 velocity=10
- joint femur_joint2: limit lower=-0.567 upper=-1.579 effort=10 velocity=10 -> lower=-1.579 upper=-0.567 effort=10 velocity=10
- joint femur_joint3: limit lower=-0.567 upper=-1.579 effort=10 velocity=10 -> lower=-1.579 upper=-0.567 effort=10 velocity=10
- joint femur_joint4: limit lower=-0.567 upper=-1.579 effort=10 velocity=10 -> lower=-1.579 upper=-0.567 effort=10 velocity=10

Commit message: control seems to be working

File: urdf/openDog_full.urdf (robot description, URDF)
Before this commit: robot opendog, 14 links, 13 joints
Joints:
- joint femur_joint1: limit lower=-1.579 upper=-0.567 effort=10 velocity=10 -> lower=-1.579 upper=-0.567 effort=5000 velocity=1.0
- joint femur_joint2: limit lower=-1.579 upper=-0.567 effort=10 velocity=10 -> lower=-1.579 upper=-0.567 effort=5000 velocity=1.0
- joint femur_joint3: limit lower=-1.579 upper=-0.567 effort=10 velocity=10 -> lower=-1.579 upper=-0.567 effort=5000 velocity=1.0
- joint femur_joint4: limit lower=-1.579 upper=-0.567 effort=10 velocity=10 -> lower=-1.579 upper=-0.567 effort=5000 velocity=1.0
- joint knee_joint_leg1: limit lower=1.352 upper=2.8715 effort=10 velocity=10 -> lower=1.352 upper=2.8715 effort=5000 velocity=1.0
- joint knee_joint_leg2: limit lower=1.352 upper=2.8715 effort=10 velocity=10 -> lower=1.352 upper=2.8715 effort=5000 velocity=1.0
- joint knee_joint_leg3: limit lower=1.352 upper=2.8715 effort=10 velocity=10 -> lower=1.352 upper=2.8715 effort=5000 velocity=1.0
- joint knee_joint_leg4: limit lower=1.352 upper=2.8715 effort=10 velocity=10 -> lower=1.352 upper=2.8715 effort=5000 velocity=1.0

Commit message: hip tube MOI and radius revised

File: urdf/openDog_full.urdf (robot description, URDF)
Before this commit: robot opendog, 14 links, 13 joints
Links:
- link hip_tube_1: mass 1 -> 0.2257; geometry collision cylinder length=0.165 radius=0.015875; visual cylinder length=0.165 radius=0.015875
- link hip_tube_2: mass 1 -> 0.2257; geometry collision cylinder length=0.165 radius=0.015875; visual cylinder length=0.165 radius=0.015875
- link hip_tube_3: mass 1 -> 0.2257; geometry collision cylinder length=0.165 radius=0.015875; visual cylinder length=0.165 radius=0.015875
- link hip_tube_4: mass 1 -> 0.2257; geometry collision cylinder length=0.165 radius=0.015875; visual cylinder length=0.165 radius=0.015875

Commit message: joint speed limit reduced

File: urdf/openDog_full.urdf (robot description, URDF)
Before this commit: robot opendog, 14 links, 13 joints
Joints:
- joint femur_joint1: limit lower=-1.579 upper=-0.567 effort=5000 velocity=1.0 -> lower=-1.579 upper=-0.567 effort=5000 velocity=0.3
- joint femur_joint2: limit lower=-1.579 upper=-0.567 effort=5000 velocity=1.0 -> lower=-1.579 upper=-0.567 effort=5000 velocity=0.3
- joint femur_joint3: limit lower=-1.579 upper=-0.567 effort=5000 velocity=1.0 -> lower=-1.579 upper=-0.567 effort=5000 velocity=0.3
- joint femur_joint4: limit lower=-1.579 upper=-0.567 effort=5000 velocity=1.0 -> lower=-1.579 upper=-0.567 effort=5000 velocity=0.3
- joint knee_joint_leg1: limit lower=1.352 upper=2.8715 effort=5000 velocity=1.0 -> lower=1.352 upper=2.8715 effort=5000 velocity=0.3
- joint knee_joint_leg2: limit lower=1.352 upper=2.8715 effort=5000 velocity=1.0 -> lower=1.352 upper=2.8715 effort=5000 velocity=0.3
- joint knee_joint_leg3: limit lower=1.352 upper=2.8715 effort=5000 velocity=1.0 -> lower=1.352 upper=2.8715 effort=5000 velocity=0.3
- joint knee_joint_leg4: limit lower=1.352 upper=2.8715 effort=5000 velocity=1.0 -> lower=1.352 upper=2.8715 effort=5000 velocity=0.3

Commit message: joint speed limit reduced: 0.05

File: urdf/openDog_full.urdf (robot description, URDF)
Before this commit: robot opendog, 14 links, 13 joints
Joints:
- joint knee_joint_leg1: limit lower=1.352 upper=2.8715 effort=5000 velocity=0.3 -> lower=1.352 upper=2.8715 effort=5000 velocity=0.05
- joint knee_joint_leg2: limit lower=1.352 upper=2.8715 effort=5000 velocity=0.3 -> lower=1.352 upper=2.8715 effort=5000 velocity=0.05
- joint knee_joint_leg3: limit lower=1.352 upper=2.8715 effort=5000 velocity=0.3 -> lower=1.352 upper=2.8715 effort=5000 velocity=0.05
- joint knee_joint_leg4: limit lower=1.352 upper=2.8715 effort=5000 velocity=0.3 -> lower=1.352 upper=2.8715 effort=5000 velocity=0.05

Commit message: joint effort and p-gain increased

File: urdf/openDog_full.urdf (robot description, URDF)
Before this commit: robot opendog, 14 links, 13 joints
Joints:
- joint femur_joint1: limit lower=-1.579 upper=-0.567 effort=5000 velocity=0.3 -> lower=-1.579 upper=-0.567 effort=8000 velocity=0.3
- joint femur_joint2: limit lower=-1.579 upper=-0.567 effort=5000 velocity=0.3 -> lower=-1.579 upper=-0.567 effort=8000 velocity=0.3
- joint femur_joint3: limit lower=-1.579 upper=-0.567 effort=5000 velocity=0.3 -> lower=-1.579 upper=-0.567 effort=8000 velocity=0.3
- joint femur_joint4: limit lower=-1.579 upper=-0.567 effort=5000 velocity=0.3 -> lower=-1.579 upper=-0.567 effort=8000 velocity=0.3
- joint knee_joint_leg1: limit lower=1.352 upper=2.8715 effort=5000 velocity=0.05 -> lower=1.352 upper=2.8715 effort=8000 velocity=0.05
- joint knee_joint_leg2: limit lower=1.352 upper=2.8715 effort=5000 velocity=0.05 -> lower=1.352 upper=2.8715 effort=8000 velocity=0.05
- joint knee_joint_leg3: limit lower=1.352 upper=2.8715 effort=5000 velocity=0.05 -> lower=1.352 upper=2.8715 effort=8000 velocity=0.05
- joint knee_joint_leg4: limit lower=1.352 upper=2.8715 effort=5000 velocity=0.05 -> lower=1.352 upper=2.8715 effort=8000 velocity=0.05

Commit message: joint velocity increased

File: urdf/openDog_full.urdf (robot description, URDF)
Before this commit: robot opendog, 14 links, 13 joints
Joints:
- joint femur_joint1: limit lower=-1.579 upper=-0.567 effort=8000 velocity=0.3 -> lower=-1.579 upper=-0.567 effort=8000 velocity=0.1
- joint femur_joint2: limit lower=-1.579 upper=-0.567 effort=8000 velocity=0.3 -> lower=-1.579 upper=-0.567 effort=8000 velocity=0.1
- joint femur_joint3: limit lower=-1.579 upper=-0.567 effort=8000 velocity=0.3 -> lower=-1.579 upper=-0.567 effort=8000 velocity=0.1
- joint femur_joint4: limit lower=-1.579 upper=-0.567 effort=8000 velocity=0.3 -> lower=-1.579 upper=-0.567 effort=8000 velocity=0.1
- joint knee_joint_leg1: limit lower=1.352 upper=2.8715 effort=8000 velocity=0.05 -> lower=1.352 upper=2.8715 effort=8000 velocity=0.1
- joint knee_joint_leg2: limit lower=1.352 upper=2.8715 effort=8000 velocity=0.05 -> lower=1.352 upper=2.8715 effort=8000 velocity=0.1
- joint knee_joint_leg3: limit lower=1.352 upper=2.8715 effort=8000 velocity=0.05 -> lower=1.352 upper=2.8715 effort=8000 velocity=0.1
- joint knee_joint_leg4: limit lower=1.352 upper=2.8715 effort=8000 velocity=0.05 -> lower=1.352 upper=2.8715 effort=8000 velocity=0.1

Commit message: extrusion weight revised

File: urdf/openDog_full.urdf (robot description, URDF)
Before this commit: robot opendog, 14 links, 13 joints
Links:
- link lower_extrusion_leg1: mass 2.224 -> 0.556
- link lower_extrusion_leg2: mass 2.224 -> 0.556
- link lower_extrusion_leg3: mass 2.224 -> 0.556
- link lower_extrusion_leg4: mass 2.224 -> 0.556
- link upper_extrusion_leg1: mass 4.036 -> 1.009
- link upper_extrusion_leg2: mass 4.036 -> 1.009
- link upper_extrusion_leg3: mass 4.036 -> 1.009
- link upper_extrusion_leg4: mass 4.036 -> 1.009

Commit message: femur joint upper limit changed

File: urdf/openDog_full.urdf (robot description, URDF)
Before this commit: robot opendog, 14 links, 13 joints
Joints:
- joint femur_joint1: limit lower=-1.579 upper=-0.567 effort=8000 velocity=0.1 -> lower=-1.579 upper=-0.3 effort=8000 velocity=0.1
- joint femur_joint2: limit lower=-1.579 upper=-0.567 effort=8000 velocity=0.1 -> lower=-1.579 upper=-0.3 effort=8000 velocity=0.1
- joint femur_joint3: limit lower=-1.579 upper=-0.567 effort=8000 velocity=0.1 -> lower=-1.579 upper=-0.3 effort=8000 velocity=0.1
- joint femur_joint4: limit lower=-1.579 upper=-0.567 effort=8000 velocity=0.1 -> lower=-1.579 upper=-0.3 effort=8000 velocity=0.1

Commit message: femur joint coordinate transformed

File: urdf/openDog_full.urdf (robot description, URDF)
Before this commit: robot opendog, 14 links, 13 joints
Joints:
- joint femur_joint1: axis 0 0 1 -> 1 0 0; limit lower=-1.579 upper=-0.3 effort=8000 velocity=0.1 -> lower=1.579 upper=0.3 effort=8000 velocity=0.1; origin xyz=-0.05 0 0 rpy=1.5708 -3.14 1.5708 -> xyz=-0.05 0 0 rpy=-3.14 0 0
- joint femur_joint2: axis 0 0 1 -> 1 0 0; limit lower=-1.579 upper=-0.3 effort=8000 velocity=0.1 -> lower=1.579 upper=0.3 effort=8000 velocity=0.1; origin xyz=0.05 0 0 rpy=1.5708 -3.14 1.5708 -> xyz=0.05 0 0 rpy=-3.14 0 0
- joint femur_joint3: axis 0 0 1 -> 1 0 0; limit lower=-1.579 upper=-0.3 effort=8000 velocity=0.1 -> lower=1.579 upper=0.3 effort=8000 velocity=0.1; origin xyz=-0.05 0 0 rpy=1.5708 -3.14 1.5708 -> xyz=-0.05 0 0 rpy=-3.14 0 0
- joint femur_joint4: axis 0 0 1 -> 1 0 0; limit lower=-1.579 upper=-0.3 effort=8000 velocity=0.1 -> lower=1.579 upper=0.3 effort=8000 velocity=0.1; origin xyz=0.05 0 0 rpy=1.5708 -3.14 1.5708 -> xyz=0.05 0 0 rpy=-3.14 0 0
- joint knee_joint_leg1: origin xyz=0 0.39 0 rpy=0 0 0 -> xyz=0 0.39 0 rpy=1.5708 1.5708 1.5708
- joint knee_joint_leg2: origin xyz=0 0.39 0 rpy=0 0 0 -> xyz=0 0.39 0 rpy=1.5708 1.5708 1.5708
- joint knee_joint_leg3: origin xyz=0 0.39 0 rpy=0 0 0 -> xyz=0 0.39 0 rpy=1.5708 1.5708 1.5708
- joint knee_joint_leg4: origin xyz=0 0.39 0 rpy=0 0 0  -> xyz=0 0.39 0 rpy=1.5708 1.5708 1.5708

Commit message: femur joint limit switched

File: urdf/openDog_full.urdf (robot description, URDF)
Before this commit: robot opendog, 14 links, 13 joints
Joints:
- joint femur_joint1: limit lower=1.579 upper=0.3 effort=8000 velocity=0.1 -> lower=0.3 upper=1.579 effort=8000 velocity=0.1

Commit message: femur upper and lower limit switched

File: urdf/openDog_full.urdf (robot description, URDF)
Before this commit: robot opendog, 14 links, 13 joints
Joints:
- joint femur_joint2: limit lower=1.579 upper=0.3 effort=8000 velocity=0.1 -> lower=0.3 upper=1.579 effort=8000 velocity=0.1
- joint femur_joint3: limit lower=1.579 upper=0.3 effort=8000 velocity=0.1 -> lower=0.3 upper=1.579 effort=8000 velocity=0.1
- joint femur_joint4: limit lower=1.579 upper=0.3 effort=8000 velocity=0.1 -> lower=0.3 upper=1.579 effort=8000 velocity=0.1

Commit message: tibia lower limit reduced

File: urdf/openDog_full.urdf (robot description, URDF)
Before this commit: robot opendog, 14 links, 13 joints
Joints:
- joint knee_joint_leg1: limit lower=1.352 upper=2.8715 effort=8000 velocity=0.1 -> lower=0.44 upper=2.8715 effort=8000 velocity=0.1
- joint knee_joint_leg2: limit lower=1.352 upper=2.8715 effort=8000 velocity=0.1 -> lower=0.44 upper=2.8715 effort=8000 velocity=0.1
- joint knee_joint_leg3: limit lower=1.352 upper=2.8715 effort=8000 velocity=0.1 -> lower=0.44 upper=2.8715 effort=8000 velocity=0.1
- joint knee_joint_leg4: limit lower=1.352 upper=2.8715 effort=8000 velocity=0.1 -> lower=0.44 upper=2.8715 effort=8000 velocity=0.1
